Commit message: shrinking smok

File: models/cartpole.urdf (robot description, URDF)
Before this commit: robot physics, 4 links, 3 joints
Joints:
- joint cart_to_smol: origin xyz=0.0 0.0 0 -> xyz=0.0 0.0 0.0
- joint pole_to_smol: origin xyz=0.0 0.0 0 -> xyz=0.0 0.0 0.0

Commit message: fixed spherical joint not moving lol

File: models/cartpole.urdf (robot description, URDF)
Before this commit: robot physics, 4 links, 3 joints
Links:
- removed link smol
Joints:
- removed joint cart_to_smol
- removed joint pole_to_smol
- added joint pole_to_cart: type spherical, parent cart, child pole, origin xyz=0.0 0.0 0.0

Commit message: mostly working, need to remove ground from carptole robot

File: models/cartpole.urdf (robot description, URDF)
Before this commit: robot physics, 3 links, 2 joints
Joints:
- joint ground_to_cart: axis 0 0 1 -> (none); limit lower=-15 upper=15 effort=1000.0 velocity=5 -> (none); type planar -> floating

Commit message: robots working

File: models/cartpole.urdf (robot description, URDF)
Before this commit: robot physics, 3 links, 2 joints
Links:
- removed link ground
Joints:
- removed joint ground_to_cart

Commit message: cleeaning urdf files

File: models/cartpole.urdf (robot description, URDF)
Before this commit: robot physics, 2 links, 1 joints
Links:
- link cart: geometry collision cylinder length=0.1 radius=0.5; visual cylinder length=0.1 radius=0.25

Commit message: fixing end conditions

File: models/cartpole.urdf (robot description, URDF)
Before this commit: robot cartpole, 2 links, 1 joints
Links:
- link pole: mass 10 -> 1; geometry collision box size=0.05 0.05 2.0; visual box size=0.05 0.05 2.0
