Commit message: param changes, bouncy walls, random posvel for blocks

File: models/block.urdf (robot description, URDF)
Before this commit: robot block, 1 links, 0 joints
Links:
- link block: mass 1 -> 10

Commit message: bigger cylenders

File: models/block.urdf (robot description, URDF)
Before this commit: robot block, 1 links, 0 joints
Links:
- link block: geometry collision cylinder length=0.1 radius=0.5; visual cylinder length=0.1 radius=0.5

File: models/cartpole.urdf (robot description, URDF)
Before this commit: robot cartpole, 2 links, 1 joints
Links:
- link cart: geometry collision cylinder length=0.1 radius=0.5; visual cylinder length=0.1 radius=0.5
- link pole: geometry collision box size=0.05 0.05 1.0; visual box size=0.05 0.05 2.0

Commit message: fixing base cartpole params

File: models/block.urdf (robot description, URDF)
Before this commit: robot block, 1 links, 0 joints
Links:
- link block: geometry collision cylinder length=0.2 radius=0.5; visual cylinder length=0.2 radius=0.5

File: models/cartpole.urdf (robot description, URDF)
Before this commit: robot cartpole, 2 links, 1 joints
Links:
- link cart: geometry collision cylinder length=0.2 radius=0.5; visual cylinder length=0.2 radius=0.5
